Commit message: added collision in urdf

File: robot_model/ground/block.urdf (robot description, URDF)
Before this commit: robot block, 1 links, 0 joints
Links:
- link baseLink: geometry collision box size=0.3 0.6 0.3; visual box size=0.3 0.6 0.3

File: robot_model/ground/stair.urdf (robot description, URDF)
Before this commit: robot stair, 2 links, 1 joints
Links:
- link baseLink: geometry collision box size=0.35 0.6 0.1; visual box size=0.35 0.6 0.1
- link secondLink: geometry collision box size=0.35 0.6 0.2; visual box size=0.35 0.6 0.2
