Commit message: draco3 stair climbing 30cm height

File: robot_model/ground/stair.urdf (robot description, URDF)
Before this commit: robot stair, 2 links, 1 joints
Links:
- link baseLink: geometry collision box size=0.35 0.6 0.15; visual box size=0.35 0.6 0.15
- link secondLink: geometry collision box size=0.35 0.6 0.3; visual box size=0.35 0.6 0.3
Joints:
- joint j0: origin xyz=0.35 0 0. rpy=0 0 0 -> xyz=0.35 0 0.0 rpy=0 0 0
