Commit message: added draco3 HandReaching test for ROM
For Frontiers submission

File: robot_model/bookcase/bookshelf.urdf (robot description, URDF)
Before this commit: robot bookcase, 9 links, 8 joints
Links:
- link back: geometry visual box size=2.1 0.02 1.6
- link leftSide: geometry visual box size=0.05 0.3 1.6
- link rightSide: geometry visual box size=0.05 0.3 1.6
- link top: geometry collision box size=2.0 0.3 0.05; visual box size=2.1 0.3 0.05
Joints:
- joint j6: origin xyz=-1 0 1.5 rpy=0 0 0 -> xyz=-1 0 1.6 rpy=0 0 0

File: robot_model/bookcase/green_can.urdf (robot description, URDF)
Before this commit: robot green_can, 1 links, 0 joints
Links:
- link can: geometry collision cylinder length=0.15 radius=0.05; visual cylinder length=0.3 radius=0.05

Commit message: added draco_ROM test
For Frontiers submission

File: robot_model/bookcase/bookshelf.urdf (robot description, URDF)
Before this commit: robot bookcase, 9 links, 8 joints
Joints:
- joint j2: origin xyz=-1 0 0.3 rpy=0 0 0 -> xyz=-1 0 0.1 rpy=0 0 0

File: robot_model/bookcase/green_can.urdf (robot description, URDF)
Before this commit: robot green_can, 1 links, 0 joints
Links:
- link can: mass 0.1 -> 2.; geometry collision cylinder length=0.2 radius=0.05; visual cylinder length=0.2 radius=0.05

File: robot_model/draco3/draco3.urdf (robot description, URDF)
Before this commit: robot draco_3, 39 links, 38 joints
Joints:
- joint l_knee_fe_jd: limit lower=-0.0872665 upper=1.52716 effort=40.85 velocity=13.35 -> lower=-0.0872665 upper=1.52716 effort=72.6 velocity=7.51
- joint l_knee_fe_jp: limit lower=-0.0872665 upper=1.52716 effort=40.85 velocity=13.35 -> lower=-0.0872665 upper=1.52716 effort=72.6 velocity=7.51
- joint r_knee_fe_jd: limit lower=-0.0872665 upper=1.52716 effort=40.85 velocity=13.35 -> lower=-0.0872665 upper=1.52716 effort=72.6 velocity=7.51
- joint r_knee_fe_jp: limit lower=-0.0872665 upper=1.52716 effort=40.85 velocity=13.35 -> lower=-0.0872665 upper=1.52716 effort=72.6 velocity=7.51
