Commit message: make atlas simulation more robust by adding utorso orientation task

File: robot_model/atlas/atlas.urdf (robot description, URDF)
Before this commit: robot multisense_sl, 34 links, 33 joints
Links:
- added link utorso_com, mass 0.001
Joints:
- added joint utorso_com_fixed: type fixed, parent utorso, child utorso_com, origin xyz=-0.0622 0.0023 0.3157 rpy=0 -0 0
